File: gardincontroller/gardincontroller.kicad_pcb (KiCad board)
At the start: 2 copper layers, 26.8 x 41 mm, 24 parts, among them J1 Conn_01x04_Male, J2 USB_C_Receptacle_USB2.0, J3 Conn_01x10_Male, J4 Conn_01x06_Male, U1 ESP32-S2-MINI-1-N4, U2 LM1117-3.3

Commit message: Fixet løse ledninger
Changed lines of the file:
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@@
   (segment (start 119.4 80.8) (end 121 79.2) (width 0.25) (layer "B.Cu") (net 4))
   (segment (start 121 79.2) (end 121.4 79.2) (width 0.25) (layer "B.Cu") (net 4))
-  (segment (start 121.3 92.7) (end 121.4 92.6) (width 0.25) (layer "B.Cu") (net 4))
   (segment (start 121.4 92.6) (end 119.4 90.6) (width 0.25) (layer "B.Cu") (net 4))
   (segment (start 111.15 98.82) (end 111.15 94.42) (width 0.25) (layer "F.Cu") (net 5))
@@
   (segment (start 123.399999 89.858515) (end 120.858515 89.858515) (width 0.25) (layer "F.Cu") (net 30))
   (segment (start 120.858515 89.858515) (end 120.8 89.8) (width 0.25) (layer "F.Cu") (net 30))
-  (segment (start 127 104.14) (end 126.66 104.14) (width 0.25) (layer "F.Cu") (net 30))
   (via (at 120.8 89.8) (size 0.8) (drill 0.4) (layers "F.Cu" "B.Cu") (net 30))
   (segment (start 124.54 104.14) (end 123.4 103) (width 0.25) (layer "B.Cu") (net 30))
@@
       )
     )
+  )
+  (zone (net 0) (net_name "") (layers F&B.Cu) (name "Antenne") (hatch edge 0.508)
+    (connect_pads (clearance 0))
+    (min_thickness 0.254)
+    (keepout (tracks not_allowed) (vias not_allowed) (pads allowed ) (copperpour not_allowed) (footprints allowed))
+    (fill (thermal_gap 0.508) (thermal_bridge_width 0.508))
+    (polygon
+      (pts
+        (xy 124 76.6)
+        (xy 109 76.6)
+        (xy 105 70.4)
+        (xy 127 70.4)
+      )
+    )
